File: Guitar Pedals/HoLo_RAT/HoLo_RAT.kicad_sch (KiCad schematic)
At the start: 35 parts, among them Q1 2n5458, U1 OP07

Commit message: [HoLo_RAT] Fixed TR pinout
Parts:
- removed Q1: 2n5458, Package_TO_SOT_THT:TO-92_Inline, symbol Simulation_SPICE:NJFET
- added Q1: 2N5458, Package_TO_SOT_THT:TO-92L_Inline, symbol Device:Q_NJFET_DSG
- C1, C12, C2, C3, C4, C8, C9: footprint Capacitor_THT:C_Disc_D4.3mm_W1.9mm_P5.00mm -> Charlie_Lee_Rhee_Custom_Parts:C_Custom_Disc_D4.3mm_W1.9mm_P5.00mm
- R1, R10, R11, R12, R2, R3, R4, R5, R6, R7, R8, R9: footprint Resistor_THT:R_Axial_DIN0207_L6.3mm_D2.5mm_P7.62mm_Horizontal -> Charlie_Lee_Rhee_Custom_Parts:R_Custom_Axial_DIN0207_L6.3mm_D2.5mm_P7.62mm_Horizontal
- R13: value 1K -> RLED; footprint Resistor_THT:R_Axial_DIN0207_L6.3mm_D2.5mm_P7.62mm_Horizontal -> Charlie_Lee_Rhee_Custom_Parts:R_Custom_Axial_DIN0207_L6.3mm_D2.5mm_P7.62mm_Horizontal
Connections:
- net 4.5V: no longer R13.1
- net 9V: now also R13.1, Q1.1 (D)
- net at C10.1, R9.1: now also Q1.2 (S)
- net at C9.2, R8.1: now also Q1.3 (G)
